File: tool/Tool_Control_PCB_Rev1/Tool_Control_PCB_Rev1.kicad_sch (KiCad schematic)
At the start: 34 parts, among them J1 2_pin_phoenix, J10 4_pin_phoenix, J11 2_pin_phoenix, J12 2_pin_phoenix, J13 Conn_01x02_Pin, J2 2_pin_phoenix, J3 Conn_02x04_Odd_Even, J4 4_pin_phoenix, J5 2_pin_phoenix, J6 Cut Trace/Jumper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

Commit message: pre review board
Parts:
- added U2, U3, U4, U5: ~, Seed_footprints:M3 bolt, symbol Seed_syms:Bolt Hole
- D1, D2, D4: value D_Schottky -> SK810L-TP

Commit message: rev 0 draft
Other:
- note added: "H-Bridge"
- note added: "Stepper Driver"
- note removed: "Driver"
- moved on the sheet: D2, D3, J12, J13, J3, R4, R5, TP7, U2, U3, U4, U5
